File: kicad/dc-modules-30kw/acdc-AC-SENSING.kicad_sch (KiCad schematic)
At the start: 95 parts

Commit message: Visual pass on the hand-placed sheets: four draughting defects fixed
End-to-end inspection at zoom found four things the wide view hides:

1. The reference designator collided with the first top pin's number on
   every multi-pin IC. The library default had been moved but the INSTANCE
   property is what renders -- fixed there, right-justified clear of the body.
2. Power pins on the top/bottom edges drew their name INSIDE the body,
   rotated, straight through the first left/right pin name (VDD over PC13 on
   the MCU). Their names are now suppressed; the net label outside already
   says V3P3 / DGND, which is standard practice on a large MCU.
3. Unbound symbol pins rendered as bare stubs that read as unfinished
   connections. Every one now carries an explicit no-connect marker.
4. Single-pin parts (M8 studs, heatsink tab) were drawn by the IC path as
   large empty rectangles. They now use a real terminal symbol -- a small
   open circle on a stub -- in both the KiCad 10 and legacy generators.

Both verifiers still 100.00% (1735/1735 pins, 608 components, 0 floating
labels, 0 overlapping symbols, 0 unclosed frames). Page PDFs and the EasyEDA
import bundle regenerated against the corrected MCU pin map.

Co-Authored-By: Claude Fable 5 <noreply@anthropic.com>
Changed lines of the file:
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@@
 	(symbol (lib_id "dc-modules:AMC1350-class") (at 140.97 44.45 0) (unit 1)
 		(exclude_from_sim no) (in_bom yes) (on_board yes) (dnp no)
-		(property "Reference" "UIVV1" (at 133.35 36.83 0) (effects (font (size 1.016 1.016)) (justify left)))
-		(property "Value" "AMC1350-class" (at 133.35 52.07 0) (effects (font (size 1.016 1.016)) (justify left)))
+		(property "Reference" "UIVV1" (at 130.81 36.83 0) (effects (font (size 1.016 1.016)) (justify right)))
+		(property "Value" "AMC1350-class" (at 130.81 52.07 0) (effects (font (size 1.016 1.016)) (justify right)))
 		(property "LCSC" "" (at 140.97 44.45 0) (effects (font (size 1.016 1.016)) (hide yes)))
 		(instances (project "dc-modules-30kw" (path "/f33d7ba5-191e-4d60-a818-2ab55f4c5e47" (reference "UIVV1") (unit 1)))))
@@
 	(symbol (lib_id "dc-modules:AMC1350-class") (at 41.910000000000004 123.19 0) (unit 1)
 		(exclude_from_sim no) (in_bom yes) (on_board yes) (dnp no)
-		(property "Reference" "UIVV2" (at 34.29 115.57000000000001 0) (effects (font (size 1.016 1.016)) (justify left)))
-		(property "Value" "AMC1350-class" (at 34.29 130.81 0) (effects (font (size 1.016 1.016)) (justify left)))
+		(property "Reference" "UIVV2" (at 31.75 115.57000000000001 0) (effects (font (size 1.016 1.016)) (justify right)))
+		(property "Value" "AMC1350-class" (at 31.75 130.81 0) (effects (font (size 1.016 1.016)) (justify right)))
 		(property "LCSC" "" (at 41.910000000000004 123.19 0) (effects (font (size 1.016 1.016)) (hide yes)))
 		(instances (project "dc-modules-30kw" (path "/f33d7ba5-191e-4d60-a818-2ab55f4c5e47" (reference "UIVV2") (unit 1)))))
@@
 	(symbol (lib_id "dc-modules:AMC1350-class") (at 204.47 123.19 0) (unit 1)
 		(exclude_from_sim no) (in_bom yes) (on_board yes) (dnp no)
-		(property "Reference" "UIVV3" (at 196.85 115.57000000000001 0) (effects (font (size 1.016 1.016)) (justify left)))
-		(property "Value" "AMC1350-class" (at 196.85 130.81 0) (effects (font (size 1.016 1.016)) (justify left)))
+		(property "Reference" "UIVV3" (at 194.31 115.57000000000001 0) (effects (font (size 1.016 1.016)) (justify right)))
+		(property "Value" "AMC1350-class" (at 194.31 130.81 0) (effects (font (size 1.016 1.016)) (justify right)))
 		(property "LCSC" "" (at 204.47 123.19 0) (effects (font (size 1.016 1.016)) (hide yes)))
 		(instances (project "dc-modules-30kw" (path "/f33d7ba5-191e-4d60-a818-2ab55f4c5e47" (reference "UIVV3") (unit 1)))))
@@
 	(symbol (lib_id "dc-modules:AMC1311-class") (at 41.910000000000004 203.2 0) (unit 1)
 		(exclude_from_sim no) (in_bom yes) (on_board yes) (dnp no)
-		(property "Reference" "UIVBP" (at 34.29 195.58 0) (effects (font (size 1.016 1.016)) (justify left)))
-		(property "Value" "AMC1311-class" (at 34.29 210.82 0) (effects (font (size 1.016 1.016)) (justify left)))
+		(property "Reference" "UIVBP" (at 31.75 195.58 0) (effects (font (size 1.016 1.016)) (justify right)))
+		(property "Value" "AMC1311-class" (at 31.75 210.82 0) (effects (font (size 1.016 1.016)) (justify right)))
 		(property "LCSC" "" (at 41.910000000000004 203.2 0) (effects (font (size 1.016 1.016)) (hide yes)))
 		(instances (project "dc-modules-30kw" (path "/f33d7ba5-191e-4d60-a818-2ab55f4c5e47" (reference "UIVBP") (unit 1)))))
@@
 	(symbol (lib_id "dc-modules:AMC1311-class") (at 205.74 203.2 0) (unit 1)
 		(exclude_from_sim no) (in_bom yes) (on_board yes) (dnp no)
-		(property "Reference" "UIVBM" (at 198.12 195.58 0) (effects (font (size 1.016 1.016)) (justify left)))
-		(property "Value" "AMC1311-class" (at 198.12 210.82 0) (effects (font (size 1.016 1.016)) (justify left)))
+		(property "Reference" "UIVBM" (at 195.58 195.58 0) (effects (font (size 1.016 1.016)) (justify right)))
+		(property "Value" "AMC1311-class" (at 195.58 210.82 0) (effects (font (size 1.016 1.016)) (justify right)))
 		(property "LCSC" "" (at 205.74 203.2 0) (effects (font (size 1.016 1.016)) (hide yes)))
 		(instances (project "dc-modules-30kw" (path "/f33d7ba5-191e-4d60-a818-2ab55f4c5e47" (reference "UIVBM") (unit 1)))))
@@
 	(symbol (lib_id "dc-modules:ISO5V-RFC-6K") (at 34.29 281.94 0) (unit 1)
 		(exclude_from_sim no) (in_bom yes) (on_board yes) (dnp no)
-		(property "Reference" "PS5AC" (at 26.67 274.32 0) (effects (font (size 1.016 1.016)) (justify left)))
-		(property "Value" "ISO5V-RFC-6K" (at 26.67 289.56 0) (effects (font (size 1.016 1.016)) (justify left)))
+		(property "Reference" "PS5AC" (at 24.13 274.32 0) (effects (font (size 1.016 1.016)) (justify right)))
+		(property "Value" "ISO5V-RFC-6K" (at 24.13 289.56 0) (effects (font (size 1.016 1.016)) (justify right)))
 		(property "LCSC" "" (at 34.29 281.94 0) (effects (font (size 1.016 1.016)) (hide yes)))
 		(instances (project "dc-modules-30kw" (path "/f33d7ba5-191e-4d60-a818-2ab55f4c5e47" (reference "PS5AC") (unit 1)))))
@@
 	(symbol (lib_id "dc-modules:ISO5V-RFC-6K") (at 81.28 281.94 0) (unit 1)
 		(exclude_from_sim no) (in_bom yes) (on_board yes) (dnp no)
-		(property "Reference" "PS5BUS" (at 73.66 274.32 0) (effects (font (size 1.016 1.016)) (justify left)))
-		(property "Value" "ISO5V-RFC-6K" (at 73.66 289.56 0) (effects (font (size 1.016 1.016)) (justify left)))
+		(property "Reference" "PS5BUS" (at 71.12 274.32 0) (effects (font (size 1.016 1.016)) (justify right)))
+		(property "Value" "ISO5V-RFC-6K" (at 71.12 289.56 0) (effects (font (size 1.016 1.016)) (justify right)))
 		(property "LCSC" "" (at 81.28 281.94 0) (effects (font (size 1.016 1.016)) (hide yes)))
 		(instances (project "dc-modules-30kw" (path "/f33d7ba5-191e-4d60-a818-2ab55f4c5e47" (reference "PS5BUS") (unit 1)))))
@@
 	(symbol (lib_id "dc-modules:TLV9061-class") (at 41.910000000000004 359.41 0) (unit 1)
 		(exclude_from_sim no) (in_bom yes) (on_board yes) (dnp no)
-		(property "Reference" "UAVB" (at 34.29 351.79 0) (effects (font (size 1.016 1.016)) (justify left)))
-		(property "Value" "TLV9061-class" (at 34.29 367.03000000000003 0) (effects (font (size 1.016 1.016)) (justify left)))
+		(property "Reference" "UAVB" (at 31.75 351.79 0) (effects (font (size 1.016 1.016)) (justify right)))
+		(property "Value" "TLV9061-class" (at 31.75 367.03000000000003 0) (effects (font (size 1.016 1.016)) (justify right)))
 		(property "LCSC" "" (at 41.910000000000004 359.41 0) (effects (font (size 1.016 1.016)) (hide yes)))
 		(instances (project "dc-modules-30kw" (path "/f33d7ba5-191e-4d60-a818-2ab55f4c5e47" (reference "UAVB") (unit 1)))))
