File: kicad/dc-modules-30kw/acdc-AUX-POWER.kicad_sch (KiCad schematic)
At the start: 44 parts

Commit message: Visual pass on the hand-placed sheets: four draughting defects fixed
End-to-end inspection at zoom found four things the wide view hides:

1. The reference designator collided with the first top pin's number on
   every multi-pin IC. The library default had been moved but the INSTANCE
   property is what renders -- fixed there, right-justified clear of the body.
2. Power pins on the top/bottom edges drew their name INSIDE the body,
   rotated, straight through the first left/right pin name (VDD over PC13 on
   the MCU). Their names are now suppressed; the net label outside already
   says V3P3 / DGND, which is standard practice on a large MCU.
3. Unbound symbol pins rendered as bare stubs that read as unfinished
   connections. Every one now carries an explicit no-connect marker.
4. Single-pin parts (M8 studs, heatsink tab) were drawn by the IC path as
   large empty rectangles. They now use a real terminal symbol -- a small
   open circle on a stub -- in both the KiCad 10 and legacy generators.

Both verifiers still 100.00% (1735/1735 pins, 608 components, 0 floating
labels, 0 overlapping symbols, 0 unclosed frames). Page PDFs and the EasyEDA
import bundle regenerated against the corrected MCU pin map.

Co-Authored-By: Claude Fable 5 <noreply@anthropic.com>
Changed lines of the file:
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@@
 	(symbol (lib_id "dc-modules:SIC-1700-1R") (at 41.910000000000004 33.02 0) (unit 1)
 		(exclude_from_sim no) (in_bom yes) (on_board yes) (dnp no)
-		(property "Reference" "QAUX" (at 34.29 24.13 0) (effects (font (size 1.016 1.016)) (justify left)))
-		(property "Value" "SIC-1700-1R" (at 34.29 41.910000000000004 0) (effects (font (size 1.016 1.016)) (justify left)))
+		(property "Reference" "QAUX" (at 31.75 24.13 0) (effects (font (size 1.016 1.016)) (justify right)))
+		(property "Value" "SIC-1700-1R" (at 31.75 41.910000000000004 0) (effects (font (size 1.016 1.016)) (justify right)))
 		(property "LCSC" "" (at 41.910000000000004 33.02 0) (effects (font (size 1.016 1.016)) (hide yes)))
 		(instances (project "dc-modules-30kw" (path "/0da9d8e0-f508-4089-a83b-54c8cf14f748" (reference "QAUX") (unit 1)))))
@@
 	(symbol (lib_id "dc-modules:XFMR-AUX-FLY-C") (at 41.910000000000004 60.96 0) (unit 1)
 		(exclude_from_sim no) (in_bom yes) (on_board yes) (dnp no)
-		(property "Reference" "TAUX" (at 34.29 45.72 0) (effects (font (size 1.016 1.016)) (justify left)))
-		(property "Value" "XFMR-AUX-FLY-C" (at 34.29 76.2 0) (effects (font (size 1.016 1.016)) (justify left)))
+		(property "Reference" "TAUX" (at 31.75 45.72 0) (effects (font (size 1.016 1.016)) (justify right)))
+		(property "Value" "XFMR-AUX-FLY-C" (at 31.75 76.2 0) (effects (font (size 1.016 1.016)) (justify right)))
 		(property "LCSC" "" (at 41.910000000000004 60.96 0) (effects (font (size 1.016 1.016)) (hide yes)))
 		(instances (project "dc-modules-30kw" (path "/0da9d8e0-f508-4089-a83b-54c8cf14f748" (reference "TAUX") (unit 1)))))
@@
 	(symbol (lib_id "dc-modules:NCP1252A") (at 93.98 46.99 0) (unit 1)
 		(exclude_from_sim no) (in_bom yes) (on_board yes) (dnp no)
-		(property "Reference" "UAUX" (at 86.36 36.83 0) (effects (font (size 1.016 1.016)) (justify left)))
-		(property "Value" "NCP1252A" (at 86.36 57.15 0) (effects (font (size 1.016 1.016)) (justify left)))
+		(property "Reference" "UAUX" (at 83.82000000000001 36.83 0) (effects (font (size 1.016 1.016)) (justify right)))
+		(property "Value" "NCP1252A" (at 83.82000000000001 57.15 0) (effects (font (size 1.016 1.016)) (justify right)))
 		(property "LCSC" "" (at 93.98 46.99 0) (effects (font (size 1.016 1.016)) (hide yes)))
 		(instances (project "dc-modules-30kw" (path "/0da9d8e0-f508-4089-a83b-54c8cf14f748" (reference "UAUX") (unit 1)))))
@@
 	(symbol (lib_id "dc-modules:TPS54202-class") (at 144.78 133.35 0) (unit 1)
 		(exclude_from_sim no) (in_bom yes) (on_board yes) (dnp no)
-		(property "Reference" "UBKA" (at 137.16 124.46000000000001 0) (effects (font (size 1.016 1.016)) (justify left)))
-		(property "Value" "TPS54202-class" (at 137.16 142.24 0) (effects (font (size 1.016 1.016)) (justify left)))
+		(property "Reference" "UBKA" (at 134.62 124.46000000000001 0) (effects (font (size 1.016 1.016)) (justify right)))
+		(property "Value" "TPS54202-class" (at 134.62 142.24 0) (effects (font (size 1.016 1.016)) (justify right)))
 		(property "LCSC" "" (at 144.78 133.35 0) (effects (font (size 1.016 1.016)) (hide yes)))
 		(instances (project "dc-modules-30kw" (path "/0da9d8e0-f508-4089-a83b-54c8cf14f748" (reference "UBKA") (unit 1)))))
@@
 	(symbol (lib_id "dc-modules:PH-4-FAN") (at 41.910000000000004 201.93 0) (unit 1)
 		(exclude_from_sim no) (in_bom yes) (on_board yes) (dnp no)
-		(property "Reference" "JFAN1" (at 34.29 193.04 0) (effects (font (size 1.016 1.016)) (justify left)))
-		(property "Value" "PH-4-FAN" (at 34.29 210.82 0) (effects (font (size 1.016 1.016)) (justify left)))
+		(property "Reference" "JFAN1" (at 31.75 193.04 0) (effects (font (size 1.016 1.016)) (justify right)))
+		(property "Value" "PH-4-FAN" (at 31.75 210.82 0) (effects (font (size 1.016 1.016)) (justify right)))
 		(property "LCSC" "" (at 41.910000000000004 201.93 0) (effects (font (size 1.016 1.016)) (hide yes)))
 		(instances (project "dc-modules-30kw" (path "/0da9d8e0-f508-4089-a83b-54c8cf14f748" (reference "JFAN1") (unit 1)))))
@@
 	(symbol (lib_id "dc-modules:PH-4-FAN") (at 92.71000000000001 201.93 0) (unit 1)
 		(exclude_from_sim no) (in_bom yes) (on_board yes) (dnp no)
-		(property "Reference" "JFAN2" (at 85.09 193.04 0) (effects (font (size 1.016 1.016)) (justify left)))
-		(property "Value" "PH-4-FAN" (at 85.09 210.82 0) (effects (font (size 1.016 1.016)) (justify left)))
+		(property "Reference" "JFAN2" (at 82.55 193.04 0) (effects (font (size 1.016 1.016)) (justify right)))
+		(property "Value" "PH-4-FAN" (at 82.55 210.82 0) (effects (font (size 1.016 1.016)) (justify right)))
 		(property "LCSC" "" (at 92.71000000000001 201.93 0) (effects (font (size 1.016 1.016)) (hide yes)))
 		(instances (project "dc-modules-30kw" (path "/0da9d8e0-f508-4089-a83b-54c8cf14f748" (reference "JFAN2") (unit 1)))))
@@
 	(symbol (lib_id "dc-modules:MICROFIT3-16") (at 153.67000000000002 214.63 0) (unit 1)
 		(exclude_from_sim no) (in_bom yes) (on_board yes) (dnp no)
-		(property "Reference" "JICA" (at 146.05 193.04 0) (effects (font (size 1.016 1.016)) (justify left)))
-		(property "Value" "MICROFIT3-16" (at 146.05 236.22 0) (effects (font (size 1.016 1.016)) (justify left)))
+		(property "Reference" "JICA" (at 143.51 193.04 0) (effects (font (size 1.016 1.016)) (justify right)))
+		(property "Value" "MICROFIT3-16" (at 143.51 236.22 0) (effects (font (size 1.016 1.016)) (justify right)))
 		(property "LCSC" "" (at 153.67000000000002 214.63 0) (effects (font (size 1.016 1.016)) (hide yes)))
 		(instances (project "dc-modules-30kw" (path "/0da9d8e0-f508-4089-a83b-54c8cf14f748" (reference "JICA") (unit 1)))))
