File: kicad/dc-modules-30kw/acdc-DC-LINK.kicad_sch (KiCad schematic)
At the start: 28 parts

Commit message: Visual pass on the hand-placed sheets: four draughting defects fixed
End-to-end inspection at zoom found four things the wide view hides:

1. The reference designator collided with the first top pin's number on
   every multi-pin IC. The library default had been moved but the INSTANCE
   property is what renders -- fixed there, right-justified clear of the body.
2. Power pins on the top/bottom edges drew their name INSIDE the body,
   rotated, straight through the first left/right pin name (VDD over PC13 on
   the MCU). Their names are now suppressed; the net label outside already
   says V3P3 / DGND, which is standard practice on a large MCU.
3. Unbound symbol pins rendered as bare stubs that read as unfinished
   connections. Every one now carries an explicit no-connect marker.
4. Single-pin parts (M8 studs, heatsink tab) were drawn by the IC path as
   large empty rectangles. They now use a real terminal symbol -- a small
   open circle on a stub -- in both the KiCad 10 and legacy generators.

Both verifiers still 100.00% (1735/1735 pins, 608 components, 0 floating
labels, 0 overlapping symbols, 0 unclosed frames). Page PDFs and the EasyEDA
import bundle regenerated against the corrected MCU pin map.

Co-Authored-By: Claude Fable 5 <noreply@anthropic.com>
Parts:
- JDCN, JDCP, JPEB: symbol dc-modules:STUD-M8 -> dc-modules:TERM_1
Changed lines of the file:
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@@
 	(generator "dc-modules kicad-gen")
 	(generator_version "10.0")
-	(paper "User" 275.59000000000003 274.32)
+	(paper "User" 275.59000000000003 248.92000000000002)
 	(title_block
 		(title "30kW ACDC 3of6 DC-LINK")
@@
 	(symbol (lib_id "dc-modules:QA01C-15S18") (at 34.29 121.92 0) (unit 1)
 		(exclude_from_sim no) (in_bom yes) (on_board yes) (dnp no)
-		(property "Reference" "PSQD" (at 26.67 114.3 0) (effects (font (size 1.016 1.016)) (justify left)))
-		(property "Value" "QA01C-15S18" (at 26.67 129.54 0) (effects (font (size 1.016 1.016)) (justify left)))
+		(property "Reference" "PSQD" (at 24.13 114.3 0) (effects (font (size 1.016 1.016)) (justify right)))
+		(property "Value" "QA01C-15S18" (at 24.13 129.54 0) (effects (font (size 1.016 1.016)) (justify right)))
 		(property "LCSC" "" (at 34.29 121.92 0) (effects (font (size 1.016 1.016)) (hide yes)))
 		(instances (project "dc-modules-30kw" (path "/ac7f6974-7f95-4087-a269-39145d43e795" (reference "PSQD") (unit 1)))))
@@
 	(symbol (lib_id "dc-modules:TAB-M4") (at 85.09 109.22 0) (unit 1)
 		(exclude_from_sim no) (in_bom yes) (on_board yes) (dnp no)
-		(property "Reference" "QDIS" (at 77.47 101.6 0) (effects (font (size 1.016 1.016)) (justify left)))
-		(property "Value" "TAB-M4" (at 77.47 116.84 0) (effects (font (size 1.016 1.016)) (justify left)))
+		(property "Reference" "QDIS" (at 74.93 101.6 0) (effects (font (size 1.016 1.016)) (justify right)))
+		(property "Value" "TAB-M4" (at 74.93 116.84 0) (effects (font (size 1.016 1.016)) (justify right)))
 		(property "LCSC" "" (at 85.09 109.22 0) (effects (font (size 1.016 1.016)) (hide yes)))
 		(instances (project "dc-modules-30kw" (path "/ac7f6974-7f95-4087-a269-39145d43e795" (reference "QDIS") (unit 1)))))
 	(symbol (lib_id "dc-modules:SIC-1200-5A") (at 92.71000000000001 129.54 0) (unit 1)
 		(exclude_from_sim no) (in_bom yes) (on_board yes) (dnp no)
-		(property "Reference" "QDISF" (at 85.09 120.65 0) (effects (font (size 1.016 1.016)) (justify left)))
-		(property "Value" "SIC-1200-5A" (at 85.09 138.43 0) (effects (font (size 1.016 1.016)) (justify left)))
+		(property "Reference" "QDISF" (at 82.55 120.65 0) (effects (font (size 1.016 1.016)) (justify right)))
+		(property "Value" "SIC-1200-5A" (at 82.55 138.43 0) (effects (font (size 1.016 1.016)) (justify right)))
 		(property "LCSC" "" (at 92.71000000000001 129.54 0) (effects (font (size 1.016 1.016)) (hide yes)))
 		(instances (project "dc-modules-30kw" (path "/ac7f6974-7f95-4087-a269-39145d43e795" (reference "QDISF") (unit 1)))))
@@
 	(symbol (lib_id "dc-modules:TLP152-class") (at 143.51 121.92 0) (unit 1)
 		(exclude_from_sim no) (in_bom yes) (on_board yes) (dnp no)
-		(property "Reference" "UQD" (at 134.62 114.3 0) (effects (font (size 1.016 1.016)) (justify left)))
-		(property "Value" "TLP152-class" (at 134.62 129.54 0) (effects (font (size 1.016 1.016)) (justify left)))
+		(property "Reference" "UQD" (at 132.08 114.3 0) (effects (font (size 1.016 1.016)) (justify right)))
+		(property "Value" "TLP152-class" (at 132.08 129.54 0) (effects (font (size 1.016 1.016)) (justify right)))
 		(property "LCSC" "" (at 143.51 121.92 0) (effects (font (size 1.016 1.016)) (hide yes)))
 		(instances (project "dc-modules-30kw" (path "/ac7f6974-7f95-4087-a269-39145d43e795" (reference "UQD") (unit 1)))))
@@
 	(global_label "DCN" (shape output) (at 255.27 106.68 0)
 		(effects (font (size 1.016 1.016)) (justify left)))
-	(rectangle (start 12.7 168.91) (end 58.42 241.3)
+	(rectangle (start 12.7 168.91) (end 35.56 215.9)
 		(stroke (width 0.254) (type dash)) (fill (type none)))
 	(text "BUS-STUDS" (at 15.24 172.72 0)
 		(effects (font (size 2.032 2.032) (bold yes)) (justify left)))
-	(symbol (lib_id "dc-modules:STUD-M8") (at 36.83 187.96 0) (unit 1)
-		(exclude_from_sim no) (in_bom yes) (on_board yes) (dnp no)
-		(property "Reference" "JDCN" (at 29.21 180.34 0) (effects (font (size 1.016 1.016)) (justify left)))
-		(property "Value" "STUD-M8" (at 29.21 195.58 0) (effects (font (size 1.016 1.016)) (justify left)))
-		(property "LCSC" "" (at 36.83 187.96 0) (effects (font (size 1.016 1.016)) (hide yes)))
+	(symbol (lib_id "dc-modules:TERM_1") (at 27.94 185.42000000000002 0) (unit 1)
+		(exclude_from_sim no) (in_bom yes) (on_board yes) (dnp no)
+		(property "Reference" "JDCN" (at 27.94 181.61 0) (effects (font (size 1.016 1.016))))
+		(property "Value" "STUD-M8" (at 27.94 189.23 0) (effects (font (size 1.016 1.016))))
+		(property "LCSC" "" (at 27.94 185.42000000000002 0) (effects (font (size 1.016 1.016)) (hide yes)))
 		(instances (project "dc-modules-30kw" (path "/ac7f6974-7f95-4087-a269-39145d43e795" (reference "JDCN") (unit 1)))))
 	(wire (pts (xy 25.4 185.42000000000002) (xy 20.32 185.42000000000002)) (stroke (width 0) (type default)))
 	(global_label "DCN" (shape input) (at 20.32 185.42000000000002 180)
 		(effects (font (size 1.016 1.016)) (justify right)))
-	(symbol (lib_id "dc-modules:STUD-M8") (at 36.83 207.01 0) (unit 1)
-		(exclude_from_sim no) (in_bom yes) (on_board yes) (dnp no)
-		(property "Reference" "JDCP" (at 29.21 199.39000000000001 0) (effects (font (size 1.016 1.016)) (justify left)))
-		(property "Value" "STUD-M8" (at 29.21 214.63 0) (effects (font (size 1.016 1.016)) (justify left)))
-		(property "LCSC" "" (at 36.83 207.01 0) (effects (font (size 1.016 1.016)) (hide yes)))
+	(symbol (lib_id "dc-modules:TERM_1") (at 27.94 195.58 0) (unit 1)
+		(exclude_from_sim no) (in_bom yes) (on_board yes) (dnp no)
+		(property "Reference" "JDCP" (at 27.94 191.77 0) (effects (font (size 1.016 1.016))))
+		(property "Value" "STUD-M8" (at 27.94 199.39000000000001 0) (effects (font (size 1.016 1.016))))
+		(property "LCSC" "" (at 27.94 195.58 0) (effects (font (size 1.016 1.016)) (hide yes)))
 		(instances (project "dc-modules-30kw" (path "/ac7f6974-7f95-4087-a269-39145d43e795" (reference "JDCP") (unit 1)))))
-	(wire (pts (xy 25.4 204.47) (xy 20.32 204.47)) (stroke (width 0) (type default)))
-	(global_label "DCP" (shape input) (at 20.32 204.47 180)
-		(effects (font (size 1.016 1.016)) (justify right)))
-	(symbol (lib_id "dc-modules:STUD-M8") (at 36.83 224.79 0) (unit 1)
-		(exclude_from_sim no) (in_bom yes) (on_board yes) (dnp no)
-		(property "Reference" "JPEB" (at 29.21 217.17000000000002 0) (effects (font (size 1.016 1.016)) (justify left)))
-		(property "Value" "STUD-M8" (at 29.21 232.41 0) (effects (font (size 1.016 1.016)) (justify left)))
-		(property "LCSC" "" (at 36.83 224.79 0) (effects (font (size 1.016 1.016)) (hide yes)))
+	(wire (pts (xy 25.4 195.58) (xy 20.32 195.58)) (stroke (width 0) (type default)))
+	(global_label "DCP" (shape input) (at 20.32 195.58 180)
+		(effects (font (size 1.016 1.016)) (justify right)))
+	(symbol (lib_id "dc-modules:TERM_1") (at 26.67 205.74 0) (unit 1)
+		(exclude_from_sim no) (in_bom yes) (on_board yes) (dnp no)
+		(property "Reference" "JPEB" (at 26.67 201.93 0) (effects (font (size 1.016 1.016))))
+		(property "Value" "STUD-M8" (at 26.67 209.55 0) (effects (font (size 1.016 1.016))))
+		(property "LCSC" "" (at 26.67 205.74 0) (effects (font (size 1.016 1.016)) (hide yes)))
 		(instances (project "dc-modules-30kw" (path "/ac7f6974-7f95-4087-a269-39145d43e795" (reference "JPEB") (unit 1)))))
-	(wire (pts (xy 25.4 222.25) (xy 20.32 222.25)) (stroke (width 0) (type default)))
-	(global_label "PE" (shape input) (at 20.32 222.25 180)
+	(wire (pts (xy 24.13 205.74) (xy 19.05 205.74)) (stroke (width 0) (type default)))
+	(global_label "PE" (shape input) (at 19.05 205.74 180)
 		(effects (font (size 1.016 1.016)) (justify right)))
 	(sheet_instances (path "/" (page "1")))
