File: kicad/dc-modules-30kw/acdc-VIENNA-PFC.kicad_sch (KiCad schematic)
At the start: 69 parts

Commit message: Visual pass on the hand-placed sheets: four draughting defects fixed
End-to-end inspection at zoom found four things the wide view hides:

1. The reference designator collided with the first top pin's number on
   every multi-pin IC. The library default had been moved but the INSTANCE
   property is what renders -- fixed there, right-justified clear of the body.
2. Power pins on the top/bottom edges drew their name INSIDE the body,
   rotated, straight through the first left/right pin name (VDD over PC13 on
   the MCU). Their names are now suppressed; the net label outside already
   says V3P3 / DGND, which is standard practice on a large MCU.
3. Unbound symbol pins rendered as bare stubs that read as unfinished
   connections. Every one now carries an explicit no-connect marker.
4. Single-pin parts (M8 studs, heatsink tab) were drawn by the IC path as
   large empty rectangles. They now use a real terminal symbol -- a small
   open circle on a stub -- in both the KiCad 10 and legacy generators.

Both verifiers still 100.00% (1735/1735 pins, 608 components, 0 floating
labels, 0 overlapping symbols, 0 unclosed frames). Page PDFs and the EasyEDA
import bundle regenerated against the corrected MCU pin map.

Co-Authored-By: Claude Fable 5 <noreply@anthropic.com>
Changed lines of the file:
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@@
 	(symbol (lib_id "dc-modules:QA01C-15S18") (at 34.29 44.45 0) (unit 1)
 		(exclude_from_sim no) (in_bom yes) (on_board yes) (dnp no)
-		(property "Reference" "PSA0G" (at 26.67 36.83 0) (effects (font (size 1.016 1.016)) (justify left)))
-		(property "Value" "QA01C-15S18" (at 26.67 52.07 0) (effects (font (size 1.016 1.016)) (justify left)))
+		(property "Reference" "PSA0G" (at 24.13 36.83 0) (effects (font (size 1.016 1.016)) (justify right)))
+		(property "Value" "QA01C-15S18" (at 24.13 52.07 0) (effects (font (size 1.016 1.016)) (justify right)))
 		(property "LCSC" "" (at 34.29 44.45 0) (effects (font (size 1.016 1.016)) (hide yes)))
 		(instances (project "dc-modules-30kw" (path "/aba155c1-ac25-4435-ad1e-bd9b82d06a2a" (reference "PSA0G") (unit 1)))))
@@
 	(symbol (lib_id "dc-modules:B3M010C075Z") (at 40.64 76.2 0) (unit 1)
 		(exclude_from_sim no) (in_bom yes) (on_board yes) (dnp no)
-		(property "Reference" "QA0A" (at 33.02 66.04 0) (effects (font (size 1.016 1.016)) (justify left)))
-		(property "Value" "B3M010C075Z" (at 33.02 86.36 0) (effects (font (size 1.016 1.016)) (justify left)))
+		(property "Reference" "QA0A" (at 30.48 66.04 0) (effects (font (size 1.016 1.016)) (justify right)))
+		(property "Value" "B3M010C075Z" (at 30.48 86.36 0) (effects (font (size 1.016 1.016)) (justify right)))
 		(property "LCSC" "" (at 40.64 76.2 0) (effects (font (size 1.016 1.016)) (hide yes)))
 		(instances (project "dc-modules-30kw" (path "/aba155c1-ac25-4435-ad1e-bd9b82d06a2a" (reference "QA0A") (unit 1)))))
@@
 	(symbol (lib_id "dc-modules:B3M010C075Z") (at 91.44 34.29 0) (unit 1)
 		(exclude_from_sim no) (in_bom yes) (on_board yes) (dnp no)
-		(property "Reference" "QA0B" (at 83.82000000000001 24.13 0) (effects (font (size 1.016 1.016)) (justify left)))
-		(property "Value" "B3M010C075Z" (at 83.82000000000001 44.45 0) (effects (font (size 1.016 1.016)) (justify left)))
+		(property "Reference" "QA0B" (at 81.28 24.13 0) (effects (font (size 1.016 1.016)) (justify right)))
+		(property "Value" "B3M010C075Z" (at 81.28 44.45 0) (effects (font (size 1.016 1.016)) (justify right)))
 		(property "LCSC" "" (at 91.44 34.29 0) (effects (font (size 1.016 1.016)) (hide yes)))
 		(instances (project "dc-modules-30kw" (path "/aba155c1-ac25-4435-ad1e-bd9b82d06a2a" (reference "QA0B") (unit 1)))))
@@
 	(symbol (lib_id "dc-modules:NSI6611") (at 143.51 52.07 0) (unit 1)
 		(exclude_from_sim no) (in_bom yes) (on_board yes) (dnp no)
-		(property "Reference" "UA0G" (at 134.62 36.83 0) (effects (font (size 1.016 1.016)) (justify left)))
-		(property "Value" "NSI6611" (at 134.62 67.31 0) (effects (font (size 1.016 1.016)) (justify left)))
+		(property "Reference" "UA0G" (at 132.08 36.83 0) (effects (font (size 1.016 1.016)) (justify right)))
+		(property "Value" "NSI6611" (at 132.08 67.31 0) (effects (font (size 1.016 1.016)) (justify right)))
 		(property "LCSC" "" (at 143.51 52.07 0) (effects (font (size 1.016 1.016)) (hide yes)))
 		(instances (project "dc-modules-30kw" (path "/aba155c1-ac25-4435-ad1e-bd9b82d06a2a" (reference "UA0G") (unit 1)))))
@@
 	(symbol (lib_id "dc-modules:QA01C-15S18") (at 34.29 138.43 0) (unit 1)
 		(exclude_from_sim no) (in_bom yes) (on_board yes) (dnp no)
-		(property "Reference" "PSB0G" (at 26.67 130.81 0) (effects (font (size 1.016 1.016)) (justify left)))
-		(property "Value" "QA01C-15S18" (at 26.67 146.05 0) (effects (font (size 1.016 1.016)) (justify left)))
+		(property "Reference" "PSB0G" (at 24.13 130.81 0) (effects (font (size 1.016 1.016)) (justify right)))
+		(property "Value" "QA01C-15S18" (at 24.13 146.05 0) (effects (font (size 1.016 1.016)) (justify right)))
 		(property "LCSC" "" (at 34.29 138.43 0) (effects (font (size 1.016 1.016)) (hide yes)))
 		(instances (project "dc-modules-30kw" (path "/aba155c1-ac25-4435-ad1e-bd9b82d06a2a" (reference "PSB0G") (unit 1)))))
@@
 	(symbol (lib_id "dc-modules:B3M010C075Z") (at 40.64 170.18 0) (unit 1)
 		(exclude_from_sim no) (in_bom yes) (on_board yes) (dnp no)
-		(property "Reference" "QB0A" (at 33.02 160.02 0) (effects (font (size 1.016 1.016)) (justify left)))
-		(property "Value" "B3M010C075Z" (at 33.02 180.34 0) (effects (font (size 1.016 1.016)) (justify left)))
+		(property "Reference" "QB0A" (at 30.48 160.02 0) (effects (font (size 1.016 1.016)) (justify right)))
+		(property "Value" "B3M010C075Z" (at 30.48 180.34 0) (effects (font (size 1.016 1.016)) (justify right)))
 		(property "LCSC" "" (at 40.64 170.18 0) (effects (font (size 1.016 1.016)) (hide yes)))
 		(instances (project "dc-modules-30kw" (path "/aba155c1-ac25-4435-ad1e-bd9b82d06a2a" (reference "QB0A") (unit 1)))))
@@
 	(symbol (lib_id "dc-modules:B3M010C075Z") (at 91.44 128.27 0) (unit 1)
 		(exclude_from_sim no) (in_bom yes) (on_board yes) (dnp no)
-		(property "Reference" "QB0B" (at 83.82000000000001 118.11 0) (effects (font (size 1.016 1.016)) (justify left)))
-		(property "Value" "B3M010C075Z" (at 83.82000000000001 138.43 0) (effects (font (size 1.016 1.016)) (justify left)))
+		(property "Reference" "QB0B" (at 81.28 118.11 0) (effects (font (size 1.016 1.016)) (justify right)))
+		(property "Value" "B3M010C075Z" (at 81.28 138.43 0) (effects (font (size 1.016 1.016)) (justify right)))
 		(property "LCSC" "" (at 91.44 128.27 0) (effects (font (size 1.016 1.016)) (hide yes)))
 		(instances (project "dc-modules-30kw" (path "/aba155c1-ac25-4435-ad1e-bd9b82d06a2a" (reference "QB0B") (unit 1)))))
@@
 	(symbol (lib_id "dc-modules:NSI6611") (at 143.51 146.05 0) (unit 1)
 		(exclude_from_sim no) (in_bom yes) (on_board yes) (dnp no)
-		(property "Reference" "UB0G" (at 134.62 130.81 0) (effects (font (size 1.016 1.016)) (justify left)))
-		(property "Value" "NSI6611" (at 134.62 161.29 0) (effects (font (size 1.016 1.016)) (justify left)))
+		(property "Reference" "UB0G" (at 132.08 130.81 0) (effects (font (size 1.016 1.016)) (justify right)))
+		(property "Value" "NSI6611" (at 132.08 161.29 0) (effects (font (size 1.016 1.016)) (justify right)))
 		(property "LCSC" "" (at 143.51 146.05 0) (effects (font (size 1.016 1.016)) (hide yes)))
 		(instances (project "dc-modules-30kw" (path "/aba155c1-ac25-4435-ad1e-bd9b82d06a2a" (reference "UB0G") (unit 1)))))
@@
 	(symbol (lib_id "dc-modules:QA01C-15S18") (at 34.29 233.68 0) (unit 1)
 		(exclude_from_sim no) (in_bom yes) (on_board yes) (dnp no)
-		(property "Reference" "PSC0G" (at 26.67 226.06 0) (effects (font (size 1.016 1.016)) (justify left)))
-		(property "Value" "QA01C-15S18" (at 26.67 241.3 0) (effects (font (size 1.016 1.016)) (justify left)))
+		(property "Reference" "PSC0G" (at 24.13 226.06 0) (effects (font (size 1.016 1.016)) (justify right)))
+		(property "Value" "QA01C-15S18" (at 24.13 241.3 0) (effects (font (size 1.016 1.016)) (justify right)))
 		(property "LCSC" "" (at 34.29 233.68 0) (effects (font (size 1.016 1.016)) (hide yes)))
 		(instances (project "dc-modules-30kw" (path "/aba155c1-ac25-4435-ad1e-bd9b82d06a2a" (reference "PSC0G") (unit 1)))))
@@
 	(symbol (lib_id "dc-modules:B3M010C075Z") (at 40.64 265.43 0) (unit 1)
 		(exclude_from_sim no) (in_bom yes) (on_board yes) (dnp no)
-		(property "Reference" "QC0A" (at 33.02 255.27 0) (effects (font (size 1.016 1.016)) (justify left)))
-		(property "Value" "B3M010C075Z" (at 33.02 275.59000000000003 0) (effects (font (size 1.016 1.016)) (justify left)))
+		(property "Reference" "QC0A" (at 30.48 255.27 0) (effects (font (size 1.016 1.016)) (justify right)))
+		(property "Value" "B3M010C075Z" (at 30.48 275.59000000000003 0) (effects (font (size 1.016 1.016)) (justify right)))
 		(property "LCSC" "" (at 40.64 265.43 0) (effects (font (size 1.016 1.016)) (hide yes)))
 		(instances (project "dc-modules-30kw" (path "/aba155c1-ac25-4435-ad1e-bd9b82d06a2a" (reference "QC0A") (unit 1)))))
@@
 	(symbol (lib_id "dc-modules:B3M010C075Z") (at 91.44 223.52 0) (unit 1)
 		(exclude_from_sim no) (in_bom yes) (on_board yes) (dnp no)
-		(property "Reference" "QC0B" (at 83.82000000000001 213.36 0) (effects (font (size 1.016 1.016)) (justify left)))
-		(property "Value" "B3M010C075Z" (at 83.82000000000001 233.68 0) (effects (font (size 1.016 1.016)) (justify left)))
+		(property "Reference" "QC0B" (at 81.28 213.36 0) (effects (font (size 1.016 1.016)) (justify right)))
+		(property "Value" "B3M010C075Z" (at 81.28 233.68 0) (effects (font (size 1.016 1.016)) (justify right)))
 		(property "LCSC" "" (at 91.44 223.52 0) (effects (font (size 1.016 1.016)) (hide yes)))
 		(instances (project "dc-modules-30kw" (path "/aba155c1-ac25-4435-ad1e-bd9b82d06a2a" (reference "QC0B") (unit 1)))))
@@
 	(symbol (lib_id "dc-modules:NSI6611") (at 143.51 241.3 0) (unit 1)
 		(exclude_from_sim no) (in_bom yes) (on_board yes) (dnp no)
-		(property "Reference" "UC0G" (at 134.62 226.06 0) (effects (font (size 1.016 1.016)) (justify left)))
-		(property "Value" "NSI6611" (at 134.62 256.54 0) (effects (font (size 1.016 1.016)) (justify left)))
+		(property "Reference" "UC0G" (at 132.08 226.06 0) (effects (font (size 1.016 1.016)) (justify right)))
+		(property "Value" "NSI6611" (at 132.08 256.54 0) (effects (font (size 1.016 1.016)) (justify right)))
 		(property "LCSC" "" (at 143.51 241.3 0) (effects (font (size 1.016 1.016)) (hide yes)))
 		(instances (project "dc-modules-30kw" (path "/aba155c1-ac25-4435-ad1e-bd9b82d06a2a" (reference "UC0G") (unit 1)))))
