File: kicad/dc-modules-30kw/dcdc-BANKS-SP.kicad_sch (KiCad schematic)
At the start: 48 parts

Commit message: Visual pass on the hand-placed sheets: four draughting defects fixed
End-to-end inspection at zoom found four things the wide view hides:

1. The reference designator collided with the first top pin's number on
   every multi-pin IC. The library default had been moved but the INSTANCE
   property is what renders -- fixed there, right-justified clear of the body.
2. Power pins on the top/bottom edges drew their name INSIDE the body,
   rotated, straight through the first left/right pin name (VDD over PC13 on
   the MCU). Their names are now suppressed; the net label outside already
   says V3P3 / DGND, which is standard practice on a large MCU.
3. Unbound symbol pins rendered as bare stubs that read as unfinished
   connections. Every one now carries an explicit no-connect marker.
4. Single-pin parts (M8 studs, heatsink tab) were drawn by the IC path as
   large empty rectangles. They now use a real terminal symbol -- a small
   open circle on a stub -- in both the KiCad 10 and legacy generators.

Both verifiers still 100.00% (1735/1735 pins, 608 components, 0 floating
labels, 0 overlapping symbols, 0 unclosed frames). Page PDFs and the EasyEDA
import bundle regenerated against the corrected MCU pin map.

Co-Authored-By: Claude Fable 5 <noreply@anthropic.com>
Changed lines of the file:
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@@
 	(symbol (lib_id "dc-modules:HFE82V-M-CLASS") (at 44.45 114.3 0) (unit 1)
 		(exclude_from_sim no) (in_bom yes) (on_board yes) (dnp no)
-		(property "Reference" "KOUT" (at 36.83 101.6 0) (effects (font (size 1.016 1.016)) (justify left)))
-		(property "Value" "HFE82V-M-CLASS" (at 36.83 127 0) (effects (font (size 1.016 1.016)) (justify left)))
+		(property "Reference" "KOUT" (at 34.29 101.6 0) (effects (font (size 1.016 1.016)) (justify right)))
+		(property "Value" "HFE82V-M-CLASS" (at 34.29 127 0) (effects (font (size 1.016 1.016)) (justify right)))
 		(property "LCSC" "" (at 44.45 114.3 0) (effects (font (size 1.016 1.016)) (hide yes)))
 		(instances (project "dc-modules-30kw" (path "/b86c33f3-6249-4515-a35f-a65ae360eb22" (reference "KOUT") (unit 1)))))
@@
 	(symbol (lib_id "dc-modules:HFE82V-M-CLASS") (at 44.45 143.51 0) (unit 1)
 		(exclude_from_sim no) (in_bom yes) (on_board yes) (dnp no)
-		(property "Reference" "KPARA" (at 36.83 130.81 0) (effects (font (size 1.016 1.016)) (justify left)))
-		(property "Value" "HFE82V-M-CLASS" (at 36.83 156.21 0) (effects (font (size 1.016 1.016)) (justify left)))
+		(property "Reference" "KPARA" (at 34.29 130.81 0) (effects (font (size 1.016 1.016)) (justify right)))
+		(property "Value" "HFE82V-M-CLASS" (at 34.29 156.21 0) (effects (font (size 1.016 1.016)) (justify right)))
 		(property "LCSC" "" (at 44.45 143.51 0) (effects (font (size 1.016 1.016)) (hide yes)))
 		(instances (project "dc-modules-30kw" (path "/b86c33f3-6249-4515-a35f-a65ae360eb22" (reference "KPARA") (unit 1)))))
@@
 	(symbol (lib_id "dc-modules:HFE82V-M-CLASS") (at 99.06 114.3 0) (unit 1)
 		(exclude_from_sim no) (in_bom yes) (on_board yes) (dnp no)
-		(property "Reference" "KPARB" (at 91.44 101.6 0) (effects (font (size 1.016 1.016)) (justify left)))
-		(property "Value" "HFE82V-M-CLASS" (at 91.44 127 0) (effects (font (size 1.016 1.016)) (justify left)))
+		(property "Reference" "KPARB" (at 88.9 101.6 0) (effects (font (size 1.016 1.016)) (justify right)))
+		(property "Value" "HFE82V-M-CLASS" (at 88.9 127 0) (effects (font (size 1.016 1.016)) (justify right)))
 		(property "LCSC" "" (at 99.06 114.3 0) (effects (font (size 1.016 1.016)) (hide yes)))
 		(instances (project "dc-modules-30kw" (path "/b86c33f3-6249-4515-a35f-a65ae360eb22" (reference "KPARB") (unit 1)))))
@@
 	(symbol (lib_id "dc-modules:HFE9-10A-1kV-M") (at 99.06 143.51 0) (unit 1)
 		(exclude_from_sim no) (in_bom yes) (on_board yes) (dnp no)
-		(property "Reference" "KPREA" (at 91.44 130.81 0) (effects (font (size 1.016 1.016)) (justify left)))
-		(property "Value" "HFE9-10A-1kV-M" (at 91.44 156.21 0) (effects (font (size 1.016 1.016)) (justify left)))
+		(property "Reference" "KPREA" (at 88.9 130.81 0) (effects (font (size 1.016 1.016)) (justify right)))
+		(property "Value" "HFE9-10A-1kV-M" (at 88.9 156.21 0) (effects (font (size 1.016 1.016)) (justify right)))
 		(property "LCSC" "" (at 99.06 143.51 0) (effects (font (size 1.016 1.016)) (hide yes)))
 		(instances (project "dc-modules-30kw" (path "/b86c33f3-6249-4515-a35f-a65ae360eb22" (reference "KPREA") (unit 1)))))
@@
 	(symbol (lib_id "dc-modules:HFE9-10A-1kV-M") (at 153.67000000000002 114.3 0) (unit 1)
 		(exclude_from_sim no) (in_bom yes) (on_board yes) (dnp no)
-		(property "Reference" "KPREB" (at 146.05 101.6 0) (effects (font (size 1.016 1.016)) (justify left)))
-		(property "Value" "HFE9-10A-1kV-M" (at 146.05 127 0) (effects (font (size 1.016 1.016)) (justify left)))
+		(property "Reference" "KPREB" (at 143.51 101.6 0) (effects (font (size 1.016 1.016)) (justify right)))
+		(property "Value" "HFE9-10A-1kV-M" (at 143.51 127 0) (effects (font (size 1.016 1.016)) (justify right)))
 		(property "LCSC" "" (at 153.67000000000002 114.3 0) (effects (font (size 1.016 1.016)) (hide yes)))
 		(instances (project "dc-modules-30kw" (path "/b86c33f3-6249-4515-a35f-a65ae360eb22" (reference "KPREB") (unit 1)))))
@@
 	(symbol (lib_id "dc-modules:HFE82V-M-CLASS") (at 153.67000000000002 143.51 0) (unit 1)
 		(exclude_from_sim no) (in_bom yes) (on_board yes) (dnp no)
-		(property "Reference" "KSER" (at 146.05 130.81 0) (effects (font (size 1.016 1.016)) (justify left)))
-		(property "Value" "HFE82V-M-CLASS" (at 146.05 156.21 0) (effects (font (size 1.016 1.016)) (justify left)))
+		(property "Reference" "KSER" (at 143.51 130.81 0) (effects (font (size 1.016 1.016)) (justify right)))
+		(property "Value" "HFE82V-M-CLASS" (at 143.51 156.21 0) (effects (font (size 1.016 1.016)) (justify right)))
 		(property "LCSC" "" (at 153.67000000000002 143.51 0) (effects (font (size 1.016 1.016)) (hide yes)))
 		(instances (project "dc-modules-30kw" (path "/b86c33f3-6249-4515-a35f-a65ae360eb22" (reference "KSER") (unit 1)))))
@@
 	(symbol (lib_id "dc-modules:SIC-1200-5A") (at 41.910000000000004 194.31 0) (unit 1)
 		(exclude_from_sim no) (in_bom yes) (on_board yes) (dnp no)
-		(property "Reference" "QDISA" (at 34.29 185.42000000000002 0) (effects (font (size 1.016 1.016)) (justify left)))
-		(property "Value" "SIC-1200-5A" (at 34.29 203.2 0) (effects (font (size 1.016 1.016)) (justify left)))
+		(property "Reference" "QDISA" (at 31.75 185.42000000000002 0) (effects (font (size 1.016 1.016)) (justify right)))
+		(property "Value" "SIC-1200-5A" (at 31.75 203.2 0) (effects (font (size 1.016 1.016)) (justify right)))
 		(property "LCSC" "" (at 41.910000000000004 194.31 0) (effects (font (size 1.016 1.016)) (hide yes)))
 		(instances (project "dc-modules-30kw" (path "/b86c33f3-6249-4515-a35f-a65ae360eb22" (reference "QDISA") (unit 1)))))
@@
 	(symbol (lib_id "dc-modules:SIC-1200-5A") (at 41.910000000000004 215.9 0) (unit 1)
 		(exclude_from_sim no) (in_bom yes) (on_board yes) (dnp no)
-		(property "Reference" "QDISB" (at 34.29 207.01 0) (effects (font (size 1.016 1.016)) (justify left)))
-		(property "Value" "SIC-1200-5A" (at 34.29 224.79 0) (effects (font (size 1.016 1.016)) (justify left)))
+		(property "Reference" "QDISB" (at 31.75 207.01 0) (effects (font (size 1.016 1.016)) (justify right)))
+		(property "Value" "SIC-1200-5A" (at 31.75 224.79 0) (effects (font (size 1.016 1.016)) (justify right)))
 		(property "LCSC" "" (at 41.910000000000004 215.9 0) (effects (font (size 1.016 1.016)) (hide yes)))
 		(instances (project "dc-modules-30kw" (path "/b86c33f3-6249-4515-a35f-a65ae360eb22" (reference "QDISB") (unit 1)))))
@@
 	(symbol (lib_id "dc-modules:VOM1271T") (at 92.71000000000001 195.58 0) (unit 1)
 		(exclude_from_sim no) (in_bom yes) (on_board yes) (dnp no)
-		(property "Reference" "UPVA" (at 85.09 185.42000000000002 0) (effects (font (size 1.016 1.016)) (justify left)))
-		(property "Value" "VOM1271T" (at 85.09 205.74 0) (effects (font (size 1.016 1.016)) (justify left)))
+		(property "Reference" "UPVA" (at 82.55 185.42000000000002 0) (effects (font (size 1.016 1.016)) (justify right)))
+		(property "Value" "VOM1271T" (at 82.55 205.74 0) (effects (font (size 1.016 1.016)) (justify right)))
 		(property "LCSC" "" (at 92.71000000000001 195.58 0) (effects (font (size 1.016 1.016)) (hide yes)))
 		(instances (project "dc-modules-30kw" (path "/b86c33f3-6249-4515-a35f-a65ae360eb22" (reference "UPVA") (unit 1)))))
@@
 	(symbol (lib_id "dc-modules:VOM1271T") (at 92.71000000000001 219.71 0) (unit 1)
 		(exclude_from_sim no) (in_bom yes) (on_board yes) (dnp no)
-		(property "Reference" "UPVB" (at 85.09 209.55 0) (effects (font (size 1.016 1.016)) (justify left)))
-		(property "Value" "VOM1271T" (at 85.09 229.87 0) (effects (font (size 1.016 1.016)) (justify left)))
+		(property "Reference" "UPVB" (at 82.55 209.55 0) (effects (font (size 1.016 1.016)) (justify right)))
+		(property "Value" "VOM1271T" (at 82.55 229.87 0) (effects (font (size 1.016 1.016)) (justify right)))
 		(property "LCSC" "" (at 92.71000000000001 219.71 0) (effects (font (size 1.016 1.016)) (hide yes)))
 		(instances (project "dc-modules-30kw" (path "/b86c33f3-6249-4515-a35f-a65ae360eb22" (reference "UPVB") (unit 1)))))
