File: kicad/dc-modules-30kw/dcdc-COMMS-HMI.kicad_sch (KiCad schematic)
At the start: 29 parts, among them SW1 TACT-6x6, SW2 TACT-6x6

Commit message: R3: verify external PDF review against datasheets; fix confirmed defects
The reviewer's headline claim -- MOSFET/driver/MCU/regulator pin numbers do
not match the real parts -- is TRUE OF THE PDFs and FALSE OF THE NETLIST.
The design is authored with logical pin ids and remapped to physical package
pins before any netlist leaves the repo; that remap was never published, so
the drawing was unfalsifiable. It is now docs/symbol-pin-map.md (107
families, 27 remapped, 407 pins). Datasheet checks confirm our physical map
MATCHES for B3M010C075Z, SG2M023120LJ, TPS54202, NCP1252A, TLV9061,
VOM1271T, TLP152. Five further claims (VAC1/VAC2 same phase, PWM stubs,
SNS_VMID, shorted shunt sense, 185.5 kHz resonance) are refuted against the
netlist -- Lr(total) is 7.0 uH = 3 leak + 4.0 trim, so fr is 140 kHz.

But the audit found six real defects we did not know about:
- CRITICAL: the GD32G553VET6 map is STM32G474-derived. FLT sits on pin 74
  (VSS) and BOOT0 on pin 100 (VDD) -- two hard shorts; SWD is on PA6/PA7.
  Open gate item A6, never closed. Blocks fabrication; no cost impact.
- NSI6611 pin 12 is RDY (open-drain, needs a pull-up), NCP1252A pin 4 is RT
  (sets fsw), TPS3430 pins 2/4 are CWD/CRST -- all were marked no-connect.
- NSI1042 pin 7 is NC on every variant, not a second GND1 (fixed here).
- AMC1311 is single-ended: pin 3 is SHTDN not VINN, and OUTN is unused, so
  the output common-mode reads as ~+/-56 V input-referred error.
- Line CT: 63.95 A rms/cell at 285 V low line exceeds its 60 A nameplate
  continuously -> 100 A class. Balance resistors need 2 W/250 V (a 1 W 2512
  is out of spec on voltage). 24 V monitor saturates at 25.74 V.
- QA01C-15S18 does not exist at MORNSUN; renamed to QA01C.

Also makes part numbers SKU-honest -- the 30 kW relay/fuse label was printed
on the 60/120 kW sheets even though price and class were already scaled.

Costs unchanged: 29,957 / 50,780 / 94,614 @10k. The one real money finding
is 120 kW cooling: 5.0 kW needs 484 CFM, and the f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
Connections:
- net DGND: no longer UCAN.7 (GND1)
Changed lines of the file:
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@@
 	(title_block
 		(title "30kW DCDC 6of6 COMMS-HMI")
-		(date "2026-09-05")
+		(date "2026-09-06")
 		(rev "D.1")
 		(company "DC-Modules — 30 kW module")
@@
 		(effects (font (size 1.016 1.016)) (justify left)))
 	(wire (pts (xy 187.96 58.42) (xy 187.96 63.5)) (stroke (width 0) (type default)))
-	(global_label "DGND" (shape input) (at 187.96 63.5 270)
+	(global_label "CGND" (shape input) (at 187.96 63.5 270)
 		(effects (font (size 1.016 1.016)) (justify left)))
 	(wire (pts (xy 190.5 58.42) (xy 190.5 63.5)) (stroke (width 0) (type default)))
@@
 	(global_label "CGND" (shape input) (at 193.04 63.5 270)
 		(effects (font (size 1.016 1.016)) (justify left)))
-	(wire (pts (xy 195.58 58.42) (xy 195.58 63.5)) (stroke (width 0) (type default)))
-	(global_label "CGND" (shape input) (at 195.58 63.5 270)
-		(effects (font (size 1.016 1.016)) (justify left)))
 	(symbol (lib_id "dc-modules:R") (at 185.42000000000002 76.2 0) (unit 1)

Commit message: Visual pass on the hand-placed sheets: four draughting defects fixed
End-to-end inspection at zoom found four things the wide view hides:

1. The reference designator collided with the first top pin's number on
   every multi-pin IC. The library default had been moved but the INSTANCE
   property is what renders -- fixed there, right-justified clear of the body.
2. Power pins on the top/bottom edges drew their name INSIDE the body,
   rotated, straight through the first left/right pin name (VDD over PC13 on
   the MCU). Their names are now suppressed; the net label outside already
   says V3P3 / DGND, which is standard practice on a large MCU.
3. Unbound symbol pins rendered as bare stubs that read as unfinished
   connections. Every one now carries an explicit no-connect marker.
4. Single-pin parts (M8 studs, heatsink tab) were drawn by the IC path as
   large empty rectangles. They now use a real terminal symbol -- a small
   open circle on a stub -- in both the KiCad 10 and legacy generators.

Both verifiers still 100.00% (1735/1735 pins, 608 components, 0 floating
labels, 0 overlapping symbols, 0 unclosed frames). Page PDFs and the EasyEDA
import bundle regenerated against the corrected MCU pin map.

Co-Authored-By: Claude Fable 5 <noreply@anthropic.com>
Changed lines of the file:
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@@
 	(symbol (lib_id "dc-modules:PH-4") (at 38.1 31.75 0) (unit 1)
 		(exclude_from_sim no) (in_bom yes) (on_board yes) (dnp no)
-		(property "Reference" "JCAN" (at 30.48 24.13 0) (effects (font (size 1.016 1.016)) (justify left)))
-		(property "Value" "PH-4" (at 30.48 39.37 0) (effects (font (size 1.016 1.016)) (justify left)))
+		(property "Reference" "JCAN" (at 27.94 24.13 0) (effects (font (size 1.016 1.016)) (justify right)))
+		(property "Value" "PH-4" (at 27.94 39.37 0) (effects (font (size 1.016 1.016)) (justify right)))
 		(property "LCSC" "" (at 38.1 31.75 0) (effects (font (size 1.016 1.016)) (hide yes)))
 		(instances (project "dc-modules-30kw" (path "/a4eae839-6dc5-4e8f-a04a-40c9eda4e492" (reference "JCAN") (unit 1)))))
@@
 	(symbol (lib_id "dc-modules:CMC-CAN-51uH") (at 41.910000000000004 53.34 0) (unit 1)
 		(exclude_from_sim no) (in_bom yes) (on_board yes) (dnp no)
-		(property "Reference" "LCAN" (at 34.29 43.18 0) (effects (font (size 1.016 1.016)) (justify left)))
-		(property "Value" "CMC-CAN-51uH" (at 34.29 63.5 0) (effects (font (size 1.016 1.016)) (justify left)))
+		(property "Reference" "LCAN" (at 31.75 43.18 0) (effects (font (size 1.016 1.016)) (justify right)))
+		(property "Value" "CMC-CAN-51uH" (at 31.75 63.5 0) (effects (font (size 1.016 1.016)) (justify right)))
 		(property "LCSC" "" (at 41.910000000000004 53.34 0) (effects (font (size 1.016 1.016)) (hide yes)))
 		(instances (project "dc-modules-30kw" (path "/a4eae839-6dc5-4e8f-a04a-40c9eda4e492" (reference "LCAN") (unit 1)))))
@@
 	(symbol (lib_id "dc-modules:ISO5V-RFC-6K") (at 88.9 44.45 0) (unit 1)
 		(exclude_from_sim no) (in_bom yes) (on_board yes) (dnp no)
-		(property "Reference" "PSCAN" (at 81.28 36.83 0) (effects (font (size 1.016 1.016)) (justify left)))
-		(property "Value" "ISO5V-RFC-6K" (at 81.28 52.07 0) (effects (font (size 1.016 1.016)) (justify left)))
+		(property "Reference" "PSCAN" (at 78.74 36.83 0) (effects (font (size 1.016 1.016)) (justify right)))
+		(property "Value" "ISO5V-RFC-6K" (at 78.74 52.07 0) (effects (font (size 1.016 1.016)) (justify right)))
 		(property "LCSC" "" (at 88.9 44.45 0) (effects (font (size 1.016 1.016)) (hide yes)))
 		(instances (project "dc-modules-30kw" (path "/a4eae839-6dc5-4e8f-a04a-40c9eda4e492" (reference "PSCAN") (unit 1)))))
@@
 	(symbol (lib_id "dc-modules:PESD1CAN") (at 144.78 33.02 0) (unit 1)
 		(exclude_from_sim no) (in_bom yes) (on_board yes) (dnp no)
-		(property "Reference" "TVSCAN" (at 137.16 24.13 0) (effects (font (size 1.016 1.016)) (justify left)))
-		(property "Value" "PESD1CAN" (at 137.16 41.910000000000004 0) (effects (font (size 1.016 1.016)) (justify left)))
+		(property "Reference" "TVSCAN" (at 134.62 24.13 0) (effects (font (size 1.016 1.016)) (justify right)))
+		(property "Value" "PESD1CAN" (at 134.62 41.910000000000004 0) (effects (font (size 1.016 1.016)) (justify right)))
 		(property "LCSC" "" (at 144.78 33.02 0) (effects (font (size 1.016 1.016)) (hide yes)))
 		(instances (project "dc-modules-30kw" (path "/a4eae839-6dc5-4e8f-a04a-40c9eda4e492" (reference "TVSCAN") (unit 1)))))
@@
 	(symbol (lib_id "dc-modules:NSI1042") (at 187.96 46.99 0) (unit 1)
 		(exclude_from_sim no) (in_bom yes) (on_board yes) (dnp no)
-		(property "Reference" "UCAN" (at 180.34 36.83 0) (effects (font (size 1.016 1.016)) (justify left)))
-		(property "Value" "NSI1042" (at 180.34 57.15 0) (effects (font (size 1.016 1.016)) (justify left)))
+		(property "Reference" "UCAN" (at 177.8 36.83 0) (effects (font (size 1.016 1.016)) (justify right)))
+		(property "Value" "NSI1042" (at 177.8 57.15 0) (effects (font (size 1.016 1.016)) (justify right)))
 		(property "LCSC" "" (at 187.96 46.99 0) (effects (font (size 1.016 1.016)) (hide yes)))
 		(instances (project "dc-modules-30kw" (path "/a4eae839-6dc5-4e8f-a04a-40c9eda4e492" (reference "UCAN") (unit 1)))))
@@
 	(symbol (lib_id "dc-modules:LED-2DIG-0.56CC") (at 41.910000000000004 125.73 0) (unit 1)
 		(exclude_from_sim no) (in_bom yes) (on_board yes) (dnp no)
-		(property "Reference" "DISP1" (at 34.29 107.95 0) (effects (font (size 1.016 1.016)) (justify left)))
-		(property "Value" "LED-2DIG-0.56CC" (at 34.29 143.51 0) (effects (font (size 1.016 1.016)) (justify left)))
+		(property "Reference" "DISP1" (at 31.75 107.95 0) (effects (font (size 1.016 1.016)) (justify right)))
+		(property "Value" "LED-2DIG-0.56CC" (at 31.75 143.51 0) (effects (font (size 1.016 1.016)) (justify right)))
 		(property "LCSC" "" (at 41.910000000000004 125.73 0) (effects (font (size 1.016 1.016)) (hide yes)))
 		(instances (project "dc-modules-30kw" (path "/a4eae839-6dc5-4e8f-a04a-40c9eda4e492" (reference "DISP1") (unit 1)))))
@@
 	(symbol (lib_id "dc-modules:S8050") (at 41.910000000000004 156.21 0) (unit 1)
 		(exclude_from_sim no) (in_bom yes) (on_board yes) (dnp no)
-		(property "Reference" "QDIG1" (at 34.29 147.32 0) (effects (font (size 1.016 1.016)) (justify left)))
-		(property "Value" "S8050" (at 34.29 165.1 0) (effects (font (size 1.016 1.016)) (justify left)))
+		(property "Reference" "QDIG1" (at 31.75 147.32 0) (effects (font (size 1.016 1.016)) (justify right)))
+		(property "Value" "S8050" (at 31.75 165.1 0) (effects (font (size 1.016 1.016)) (justify right)))
 		(property "LCSC" "" (at 41.910000000000004 156.21 0) (effects (font (size 1.016 1.016)) (hide yes)))
 		(instances (project "dc-modules-30kw" (path "/a4eae839-6dc5-4e8f-a04a-40c9eda4e492" (reference "QDIG1") (unit 1)))))
@@
 	(symbol (lib_id "dc-modules:S8050") (at 93.98 116.84 0) (unit 1)
 		(exclude_from_sim no) (in_bom yes) (on_board yes) (dnp no)
-		(property "Reference" "QDIG2" (at 86.36 107.95 0) (effects (font (size 1.016 1.016)) (justify left)))
-		(property "Value" "S8050" (at 86.36 125.73 0) (effects (font (size 1.016 1.016)) (justify left)))
+		(property "Reference" "QDIG2" (at 83.82000000000001 107.95 0) (effects (font (size 1.016 1.016)) (justify right)))
+		(property "Value" "S8050" (at 83.82000000000001 125.73 0) (effects (font (size 1.016 1.016)) (justify right)))
 		(property "LCSC" "" (at 93.98 116.84 0) (effects (font (size 1.016 1.016)) (hide yes)))
 		(instances (project "dc-modules-30kw" (path "/a4eae839-6dc5-4e8f-a04a-40c9eda4e492" (reference "QDIG2") (unit 1)))))
@@
 	(symbol (lib_id "dc-modules:74HC595") (at 144.78 142.24 0) (unit 1)
 		(exclude_from_sim no) (in_bom yes) (on_board yes) (dnp no)
-		(property "Reference" "USR1" (at 137.16 120.65 0) (effects (font (size 1.016 1.016)) (justify left)))
-		(property "Value" "74HC595" (at 137.16 163.83 0) (effects (font (size 1.016 1.016)) (justify left)))
+		(property "Reference" "USR1" (at 134.62 120.65 0) (effects (font (size 1.016 1.016)) (justify right)))
+		(property "Value" "74HC595" (at 134.62 163.83 0) (effects (font (size 1.016 1.016)) (justify right)))
 		(property "LCSC" "" (at 144.78 142.24 0) (effects (font (size 1.016 1.016)) (hide yes)))
 		(instances (project "dc-modules-30kw" (path "/a4eae839-6dc5-4e8f-a04a-40c9eda4e492" (reference "USR1") (unit 1)))))
