File: kicad/dc-modules-30kw/dcdc-LLC-LEGS.kicad_sch (KiCad schematic)
At the start: 78 parts, among them Q1H SG2M023120LJ, Q1L SG2M023120LJ, Q2H SG2M023120LJ, Q2L SG2M023120LJ, Q3H SG2M023120LJ, Q3L SG2M023120LJ, U1H NSI6611, U1L NSI6611, U2H NSI6611, U2L NSI6611, U3H NSI6611, U3L NSI6611

Commit message: Visual pass on the hand-placed sheets: four draughting defects fixed
End-to-end inspection at zoom found four things the wide view hides:

1. The reference designator collided with the first top pin's number on
   every multi-pin IC. The library default had been moved but the INSTANCE
   property is what renders -- fixed there, right-justified clear of the body.
2. Power pins on the top/bottom edges drew their name INSIDE the body,
   rotated, straight through the first left/right pin name (VDD over PC13 on
   the MCU). Their names are now suppressed; the net label outside already
   says V3P3 / DGND, which is standard practice on a large MCU.
3. Unbound symbol pins rendered as bare stubs that read as unfinished
   connections. Every one now carries an explicit no-connect marker.
4. Single-pin parts (M8 studs, heatsink tab) were drawn by the IC path as
   large empty rectangles. They now use a real terminal symbol -- a small
   open circle on a stub -- in both the KiCad 10 and legacy generators.

Both verifiers still 100.00% (1735/1735 pins, 608 components, 0 floating
labels, 0 overlapping symbols, 0 unclosed frames). Page PDFs and the EasyEDA
import bundle regenerated against the corrected MCU pin map.

Co-Authored-By: Claude Fable 5 <noreply@anthropic.com>
Parts:
- JDCN, JDCP, JPEB: symbol dc-modules:STUD-M8 -> dc-modules:TERM_1
Other:
- moved on the sheet: C1HB1, C1HB2, C1HBL, C1LB1, C1LB2, C1LBL, C2HB1, C2HB2, C2HBL, C2LB1, C2LB2, C2LBL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
