File: kicad/dc-modules-30kw/dcdc-LLC-TANKS.kicad_sch (KiCad schematic)
At the start: 60 parts, among them T1 XFMR-LLC-10K, T2 XFMR-LLC-10K, T3 XFMR-LLC-10K

Commit message: Visual pass on the hand-placed sheets: four draughting defects fixed
End-to-end inspection at zoom found four things the wide view hides:

1. The reference designator collided with the first top pin's number on
   every multi-pin IC. The library default had been moved but the INSTANCE
   property is what renders -- fixed there, right-justified clear of the body.
2. Power pins on the top/bottom edges drew their name INSIDE the body,
   rotated, straight through the first left/right pin name (VDD over PC13 on
   the MCU). Their names are now suppressed; the net label outside already
   says V3P3 / DGND, which is standard practice on a large MCU.
3. Unbound symbol pins rendered as bare stubs that read as unfinished
   connections. Every one now carries an explicit no-connect marker.
4. Single-pin parts (M8 studs, heatsink tab) were drawn by the IC path as
   large empty rectangles. They now use a real terminal symbol -- a small
   open circle on a stub -- in both the KiCad 10 and legacy generators.

Both verifiers still 100.00% (1735/1735 pins, 608 components, 0 floating
labels, 0 overlapping symbols, 0 unclosed frames). Page PDFs and the EasyEDA
import bundle regenerated against the corrected MCU pin map.

Co-Authored-By: Claude Fable 5 <noreply@anthropic.com>
Changed lines of the file:
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@@
 	(symbol (lib_id "dc-modules:XFMR-LLC-10K") (at 41.910000000000004 38.1 0) (unit 1)
 		(exclude_from_sim no) (in_bom yes) (on_board yes) (dnp no)
-		(property "Reference" "T1" (at 34.29 24.13 0) (effects (font (size 1.016 1.016)) (justify left)))
-		(property "Value" "XFMR-LLC-10K" (at 34.29 52.07 0) (effects (font (size 1.016 1.016)) (justify left)))
+		(property "Reference" "T1" (at 31.75 24.13 0) (effects (font (size 1.016 1.016)) (justify right)))
+		(property "Value" "XFMR-LLC-10K" (at 31.75 52.07 0) (effects (font (size 1.016 1.016)) (justify right)))
 		(property "LCSC" "" (at 41.910000000000004 38.1 0) (effects (font (size 1.016 1.016)) (hide yes)))
 		(instances (project "dc-modules-30kw" (path "/90783d18-0d00-41fb-adf8-d7610a152fdb" (reference "T1") (unit 1)))))
@@
 	(symbol (lib_id "dc-modules:XFMR-LLC-10K") (at 41.910000000000004 116.84 0) (unit 1)
 		(exclude_from_sim no) (in_bom yes) (on_board yes) (dnp no)
-		(property "Reference" "T2" (at 34.29 102.87 0) (effects (font (size 1.016 1.016)) (justify left)))
-		(property "Value" "XFMR-LLC-10K" (at 34.29 130.81 0) (effects (font (size 1.016 1.016)) (justify left)))
+		(property "Reference" "T2" (at 31.75 102.87 0) (effects (font (size 1.016 1.016)) (justify right)))
+		(property "Value" "XFMR-LLC-10K" (at 31.75 130.81 0) (effects (font (size 1.016 1.016)) (justify right)))
 		(property "LCSC" "" (at 41.910000000000004 116.84 0) (effects (font (size 1.016 1.016)) (hide yes)))
 		(instances (project "dc-modules-30kw" (path "/90783d18-0d00-41fb-adf8-d7610a152fdb" (reference "T2") (unit 1)))))
@@
 	(symbol (lib_id "dc-modules:XFMR-LLC-10K") (at 41.910000000000004 194.31 0) (unit 1)
 		(exclude_from_sim no) (in_bom yes) (on_board yes) (dnp no)
-		(property "Reference" "T3" (at 34.29 180.34 0) (effects (font (size 1.016 1.016)) (justify left)))
-		(property "Value" "XFMR-LLC-10K" (at 34.29 208.28 0) (effects (font (size 1.016 1.016)) (justify left)))
+		(property "Reference" "T3" (at 31.75 180.34 0) (effects (font (size 1.016 1.016)) (justify right)))
+		(property "Value" "XFMR-LLC-10K" (at 31.75 208.28 0) (effects (font (size 1.016 1.016)) (justify right)))
 		(property "LCSC" "" (at 41.910000000000004 194.31 0) (effects (font (size 1.016 1.016)) (hide yes)))
 		(instances (project "dc-modules-30kw" (path "/90783d18-0d00-41fb-adf8-d7610a152fdb" (reference "T3") (unit 1)))))
