File: kicad/dc-modules-30kw/dcdc-OUTPUT-SENSING.kicad_sch (KiCad schematic)
At the start: 58 parts

Commit message: Visual pass on the hand-placed sheets: four draughting defects fixed
End-to-end inspection at zoom found four things the wide view hides:

1. The reference designator collided with the first top pin's number on
   every multi-pin IC. The library default had been moved but the INSTANCE
   property is what renders -- fixed there, right-justified clear of the body.
2. Power pins on the top/bottom edges drew their name INSIDE the body,
   rotated, straight through the first left/right pin name (VDD over PC13 on
   the MCU). Their names are now suppressed; the net label outside already
   says V3P3 / DGND, which is standard practice on a large MCU.
3. Unbound symbol pins rendered as bare stubs that read as unfinished
   connections. Every one now carries an explicit no-connect marker.
4. Single-pin parts (M8 studs, heatsink tab) were drawn by the IC path as
   large empty rectangles. They now use a real terminal symbol -- a small
   open circle on a stub -- in both the KiCad 10 and legacy generators.

Both verifiers still 100.00% (1735/1735 pins, 608 components, 0 floating
labels, 0 overlapping symbols, 0 unclosed frames). Page PDFs and the EasyEDA
import bundle regenerated against the corrected MCU pin map.

Co-Authored-By: Claude Fable 5 <noreply@anthropic.com>
Parts:
- JOUTN, JOUTP: symbol dc-modules:STUD-M8 -> dc-modules:TERM_1
Other:
- moved on the sheet: COF1, COF2, CYO1, CYO2, RSHO
